File: Oscillator.kicad_sch (KiCad schematic)
At the start: 11 parts, among them J1 Conn_01x01, J2 Conn_01x01, J3 Conn_01x01, J4 Conn_01x01, U1 74HC04, Y1 10 MHz

Commit message: routed all signals
Parts:
- Y1: footprint Crystal:Crystal_SMD_HC49-SD -> Crystal:Crystal_HC49-U_Vertical
Changed lines of the file:
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@@
       (effects (font (size 1.27 1.27)))
     )
-    (property "Footprint" "Crystal:Crystal_SMD_HC49-SD" (at 55.88 101.6 0)
+    (property "Footprint" "Crystal:Crystal_HC49-U_Vertical" (at 55.88 101.6 0)
       (effects (font (size 1.27 1.27)) hide)
     )
